Commit message: minor fix

File: src/my_robot_description/urdf/my_robot.urdf.xacro (robot description, xacro)
@@ -1,7 +1,4 @@
 <?xml version="1.0"?>
 <robot name="my_robot" xmlns:xacro="http://www.ros.org/wiki/xacro">
-    <!-- ========================= -->
-    <!-- Properties                -->
-    <!-- ========================= -->
     <xacro:property name="base_length" value="0.2" />
     <xacro:property name="base_width" value="0.15" />
@@ -12,12 +9,6 @@
     <xacro:property name="PI" value="3.141592653589793" />
     <xacro:property name="camera_side_length" value="0.03" />
-    <!-- ========================= -->
-    <!-- Includes                  -->
-    <!-- ========================= -->
     <xacro:include filename="$(find my_robot_description)/urdf/common_properties.xacro" />
     <xacro:include filename="$(find my_robot_description)/urdf/gazebo_plugins.xacro" />
-    <!-- ========================= -->
-    <!-- Materials                 -->
-    <!-- ========================= -->
     <material name="green">
         <color rgba="0 0.6 0 1" />
@@ -32,7 +23,4 @@
         <color rgba="0 0 1 1" />
     </material>
-    <!-- ========================= -->
-    <!-- Camera                    -->
-    <!-- ========================= -->
     <link name="camera_link">
         <xacro:box_inertia
@@ -54,7 +42,4 @@
         </visual>
     </link>
-    <!-- ========================= -->
-    <!-- Base                      -->
-    <!-- ========================= -->
     <link name="base_link">
         <xacro:box_inertia
@@ -85,10 +70,6 @@
         </visual>
     </link>
-    <!-- ========================= -->
-    <!-- Left Wheel                -->
-    <!-- ========================= -->
     <link name="left_wheel_link">
         <visual>
-            <!-- Rotate cylinder so its axis is along Y -->
             <origin
                 xyz="0 0 0"
@@ -119,11 +100,6 @@
              />
     </link>
-    <!-- ========================= -->
-    <!-- Right Wheel               -->
-    <!-- ========================= -->
     <link name="right_wheel_link">
-green
-        <visual>
-            <!-- Rotate cylinder so its axis is along Y -->
+        <visual>
             <origin
                 xyz="0 0 0"
@@ -153,7 +129,4 @@
             o_rpy="0 0 0" />
     </link>
-    <!-- ========================= -->
-    <!-- Caster Wheel              -->
-    <!-- ========================= -->
     <link name="caster_wheel_link">
         <xacro:sphere_inertia
@@ -182,11 +155,5 @@
         </visual>
     </link>
-    <!-- ========================= -->
-    <!-- Base Footprint             -->
-    <!-- ========================= -->
     <link name="base_footprint" />
-    <!-- ========================= -->
-    <!-- Camera Joint              -->
-    <!-- ========================= -->
     <joint name="base_camera_joint" type="fixed">
         <parent link="base_link" />
@@ -196,7 +163,4 @@
             rpy="0 0 0" />
     </joint>
-    <!-- ========================= -->
-    <!-- Left Wheel Joint          -->
-    <!-- ========================= -->
     <joint name="left_wheel_joint" type="continuous">
         <parent link="base_link" />
@@ -207,7 +171,4 @@
         <axis xyz="0 1 0" />
     </joint>
-    <!-- ========================= -->
-    <!-- Right Wheel Joint         -->
-    <!-- ========================= -->
     <joint name="right_wheel_joint" type="continuous">
         <parent link="base_link" />
@@ -218,7 +179,4 @@
         <axis xyz="0 1 0" />
     </joint>
-    <!-- ========================= -->
-    <!-- Caster Joint              -->
-    <!-- ========================= -->
     <joint name="base_caster_wheel_joint" type="fixed">
         <parent link="base_link" />
@@ -228,7 +186,4 @@
             rpy="0 0 0" />
     </joint>
-    <!-- ========================= -->
-    <!-- Base Joint                -->
-    <!-- ========================= -->
     <joint name="base_joint" type="fixed">
         <parent link="base_footprint" />
@@ -238,7 +193,4 @@
             rpy="0 0 0" />
     </joint>
-    <!-- ========================= -->
-    <!-- Gazebo Pose Publisher     -->
-    <!-- ========================= -->
     <gazebo>
         <plugin
